File: Potentiostat.kicad_pcb (KiCad board)
At the start: 2 copper layers, 42 parts

Commit message: Update Potentiostat.kicad_pcb
Parts:
- added ?: , DEFAULT, F.Cu at (52.5, 172.7)
- added IC1: LMP7702MA_NOPB, SOIC127P600X175-8N, F.Cu at (162.7, 114.9)
- added IC2: MAX4617ESE+, SOIC127P600X175-16N, F.Cu at (126.3, 99.5)
- added IC3: AMS1117-5.0, SOT229P700X180-4N, F.Cu at (138.0, 78.3)
- added IC4: TEENSY3.2, TEENSY32, F.Cu at (122.5, 125.7)
- added IC5: LMP7702MA_NOPB, SOIC127P600X175-8N, F.Cu at (159.7, 90.8)
- added IC6: LMP7721MA_NOPB, SOIC127P600X175-8N, F.Cu at (148.1, 99.5)
- added JP1: , KF2EDGK5.08-LI-2P, F.Cu at (115.0, 84.9)
- added JP2: , KF128-5.08-3P, F.Cu at (170.3, 91.7)
- added PS1: TPS60403DBVR, SOT95P280X145-5N, F.Cu at (162.7, 78.1)
- added SW1: KET_7X7, KFT DIP-7X7, F.Cu at (125.3, 78.5)
- C1, C3, C4, C6: footprint Capacitor_SMD:C_0805_2012Metric -> 1608[0603]
- C10, C11, C12, C13, C15, C16, C17, C18, C19, C2, C20, C21, C22, C23, C5, C7, C8, C9: footprint Capacitor_SMD:C_0805_2012Metric -> CAPC2012X130N
- C14, C24: footprint Capacitor_SMD:C_1206_3216Metric -> CAPC2012X130N
- LED1: footprint LED_SMD:LED_0805_2012Metric -> E6C1206QBAC1UDA
- R1, R10, R11, R12, R13, R15, R16, R2, R3, R4, R5, R6, R7, R8: footprint Resistor_SMD:R_0805_2012Metric -> RESC2012X65N
- R14, R17: footprint Resistor_SMD:R_0805_2012Metric -> RESC3216X75N
- R9: footprint Resistor_SMD:R_0805_2012Metric -> RESC6331X75N; moved to B.Cu
- moved C6 101.4 mm to (170.7, 122.6)
- moved C5 94.9 mm to (174.1, 122.3)
- moved C2 93.5 mm to (174.2, 108.2)
- moved C3 91.3 mm to (174.4, 113.9)
- moved LED1 90.9 mm to (164.5, 123.8)
- moved R6 88.1 mm to (168.8, 126.1)
- moved C4 86.1 mm to (157.3, 118.1)
- moved R5 82.1 mm to (170.0, 114.4)
- moved R7 81.4 mm to (168.7, 119.5)
- moved R2 80.5 mm to (168.9, 109.0)
- moved R9 78.9 mm to (157.8, 125.0)
- moved C1 77.4 mm to (163.0, 109.9)
- moved C16 76.2 mm to (169.1, 76.7)
- moved R3 69.5 mm to (161.8, 106.8)
- moved C17 67.2 mm to (162.6, 98.1)
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Routing:
- net +5: track 0.00 -> 974.4 mm, vias 0 -> 13
- net /WORKING: track 0.00 -> 86.8 mm, vias 0 -> 2
- net Net-(IC2-Pad10): track 0.00 -> 34.2 mm
- net /COUNTER: track 0.00 -> 27.1 mm, vias 0 -> 1
- net Net-(IC2-Pad11): track 0.00 -> 25.7 mm
- net Net-(IC2-Pad9): track 0.00 -> 24.0 mm
- net /REFERENCE: track 0.00 -> 18.0 mm, vias 0 -> 1
- net Net-(JP1-Pad1): track 0.00 -> 15.0 mm
- net Net-(JP1-Pad2): track 0.00 -> 15.0 mm
- added copper zone on B.Cu, net (none)
Other:
- board text added: "C1"
- board text added: "C10"
- board text added: "C11"
- board text added: "C12"
- board text added: "C13"
- board text added: "C14"
- board text added: "C15"
- board text added: "C16"
- board text added: "C17"
- board text added: "C18"
- board text added: "C19"
- board text added: "C2"
- board text added: "C20"
- board text added: "C21"
- board text added: "C22"
- board text added: "C23"
- board text added: "C24"
- board text added: "C3"
- board text added: "C4"
- board text added: "C5"
- board text added: "C6"
- board text added: "C7"
- board text added: "C8"
- board text added: "C9"
- board text added: "IC1"
- board text added: "IC2"
- board text added: "IC3"
- board text added: "IC4"
- board text added: "IC5"
- board text added: "IC6"
- board text added: "JP1"
- board text added: "JP2"
- board text added: "LED1"
- board text added: "PS1"
- board text added: "Potentiiator V2.0 16/11/22"
- board text added: "R1"
- board text added: "R10"
- board text added: "R11"
- board text added: "R12"
- board text added: "R13"
- board text added: "R14"
- board text added: "R15"
- board text added: "R16"
- board text added: "R17"
- board text added: "R2"
- board text added: "R3"
- board text added: "R4"
- board text added: "R5"
- board text added: "R6"
- board text added: "R7"
- board text added: "R8"
- board text added: "R9"
- board text added: "SW1"
