File: Potentiostat.kicad_sch (KiCad schematic)
At the start: 52 parts, among them IC1 LMP7702MA_NOPB, IC2 MAX4617ESE+, IC3 AMS1117-5.0, IC4 TEENSY3.2, IC5 LMP7702MA_NOPB, IC6 LMP7721MA_NOPB, SW1 KET_7X7

Commit message: Update Potentiostat.kicad_sch
Parts:
- IC1, IC5, IC6: footprint (none) -> PCBlibrary:SOIC127P600X175-8N
- IC2: footprint (none) -> PCBlibrary:SOIC127P600X175-16N
- IC3: footprint (none) -> PCBlibrary:SOT229P700X180-4N
- IC4: footprint (none) -> PCBlibrary:TEENSY32
- JP1: footprint (none) -> PCBlibrary:KF2EDGK5.08-LI-2P
- JP2: footprint (none) -> PCBlibrary:KF128-5.08-3P
- PS1: footprint (none) -> PCBlibrary:SOT95P280X145-5N
- SW1: footprint (none) -> PCBlibrary:KFT DIP-7X7
Changed lines of the file:
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@@
       (effects (font (size 1.524 1.524)))
     )
-    (property "Footprint" "" (id 2) (at 107.95 106.68 0)
+    (property "Footprint" "PCBlibrary:KFT DIP-7X7" (id 2) (at 107.95 106.68 0)
       (effects (font (size 1.524 1.524)) hide)
     )
@@
       (effects (font (size 1.524 1.524)))
     )
-    (property "Footprint" "" (id 2) (at 57.15 54.61 0)
+    (property "Footprint" "PCBlibrary:SOIC127P600X175-8N" (id 2) (at 57.15 54.61 0)
       (effects (font (size 1.524 1.524)) hide)
     )
@@
       (effects (font (size 1.524 1.524)))
     )
-    (property "Footprint" "" (id 2) (at 257.81 100.33 0)
+    (property "Footprint" "PCBlibrary:SOIC127P600X175-16N" (id 2) (at 257.81 100.33 0)
       (effects (font (size 1.524 1.524)) hide)
     )
@@
       (effects (font (size 1.524 1.524)))
     )
-    (property "Footprint" "" (id 2) (at 193.04 113.03 0)
+    (property "Footprint" "PCBlibrary:SOIC127P600X175-8N" (id 2) (at 193.04 113.03 0)
       (effects (font (size 1.524 1.524)) hide)
     )
@@
       (effects (font (size 1.524 1.524)) (justify left))
     )
-    (property "Footprint" "" (id 2) (at 127 109.22 0)
+    (property "Footprint" "PCBlibrary:KF2EDGK5.08-LI-2P" (id 2) (at 127 109.22 0)
       (effects (font (size 1.524 1.524)) hide)
     )
@@
       (effects (font (size 1.524 1.524)))
     )
-    (property "Footprint" "" (id 2) (at 287.02 154.94 0)
+    (property "Footprint" "PCBlibrary:SOIC127P600X175-8N" (id 2) (at 287.02 154.94 0)
       (effects (font (size 1.524 1.524)) hide)
     )
@@
       (effects (font (size 1.524 1.524)) (justify left))
     )
-    (property "Footprint" "" (id 2) (at 233.68 163.83 0)
+    (property "Footprint" "PCBlibrary:KF128-5.08-3P" (id 2) (at 233.68 163.83 0)
       (effects (font (size 1.524 1.524)) hide)
     )
@@
       (effects (font (size 1.524 1.524)))
     )
-    (property "Footprint" "" (id 2) (at 353.06 105.41 0)
+    (property "Footprint" "PCBlibrary:TEENSY32" (id 2) (at 353.06 105.41 0)
       (effects (font (size 1.524 1.524)) hide)
     )
@@
       (effects (font (size 1.524 1.524)))
     )
-    (property "Footprint" "" (id 2) (at 46.99 177.8 0)
+    (property "Footprint" "PCBlibrary:SOT95P280X145-5N" (id 2) (at 46.99 177.8 0)
       (effects (font (size 1.524 1.524)) hide)
     )
@@
       (effects (font (size 1.524 1.524)))
     )
-    (property "Footprint" "" (id 2) (at 58.42 144.78 0)
+    (property "Footprint" "PCBlibrary:SOT229P700X180-4N" (id 2) (at 58.42 144.78 0)
       (effects (font (size 1.524 1.524)) hide)
     )
@@
     )
     (path "/27241ce6-87a4-4b75-9057-7c169aa0d907"
-      (reference "IC1") (unit 1) (value "LMP7702MA_NOPB") (footprint "")
+      (reference "IC1") (unit 1) (value "LMP7702MA_NOPB") (footprint "PCBlibrary:SOIC127P600X175-8N")
     )
     (path "/3e4bde83-e996-45f7-b1bc-1b8a64e2708e"
-      (reference "IC2") (unit 1) (value "MAX4617ESE+") (footprint "")
+      (reference "IC2") (unit 1) (value "MAX4617ESE+") (footprint "PCBlibrary:SOIC127P600X175-16N")
     )
     (path "/d03f860f-39cf-4972-9162-2b86d24bee2a"
-      (reference "IC3") (unit 1) (value "AMS1117-5.0") (footprint "")
+      (reference "IC3") (unit 1) (value "AMS1117-5.0") (footprint "PCBlibrary:SOT229P700X180-4N")
     )
     (path "/ad37a0f2-2777-4a00-8a2b-c8b988e076cc"
-      (reference "IC4") (unit 1) (value "TEENSY3.2") (footprint "")
+      (reference "IC4") (unit 1) (value "TEENSY3.2") (footprint "PCBlibrary:TEENSY32")
     )
     (path "/549b8fd8-2213-4d06-9b16-23145aacb5fb"
-      (reference "IC5") (unit 1) (value "LMP7702MA_NOPB") (footprint "")
+      (reference "IC5") (unit 1) (value "LMP7702MA_NOPB") (footprint "PCBlibrary:SOIC127P600X175-8N")
     )
     (path "/a6ada26d-f62c-49ab-a6cd-340f1407a9fe"
-      (reference "IC6") (unit 1) (value "LMP7721MA_NOPB") (footprint "")
+      (reference "IC6") (unit 1) (value "LMP7721MA_NOPB") (footprint "PCBlibrary:SOIC127P600X175-8N")
     )
     (path "/61829e24-a2df-4c2d-ba21-9700d7ef336d"
-      (reference "JP1") (unit 1) (value " ") (footprint "")
+      (reference "JP1") (unit 1) (value " ") (footprint "PCBlibrary:KF2EDGK5.08-LI-2P")
     )
     (path "/ab6ab3e1-e933-448c-b029-dcb822cbac82"
-      (reference "JP2") (unit 1) (value " ") (footprint "")
+      (reference "JP2") (unit 1) (value " ") (footprint "PCBlibrary:KF128-5.08-3P")
     )
     (path "/685157d7-e988-4870-bdc0-901fbf1efcb1"
@@
     )
     (path "/c9173087-412f-4baa-98c1-c92856ec258f"
-      (reference "PS1") (unit 1) (value "TPS60403DBVR") (footprint "")
+      (reference "PS1") (unit 1) (value "TPS60403DBVR") (footprint "PCBlibrary:SOT95P280X145-5N")
     )
     (path "/01b49f4d-13e7-4cff-b16b-a7b8c6fb7c2a"
@@
     )
     (path "/260c73f3-646c-41eb-9cc5-c5d58e65a37b"
-      (reference "SW1") (unit 1) (value "KET_7X7") (footprint "")
-    )
-  )
+      (reference "SW1") (unit 1) (value "KET_7X7") (footprint "PCBlibrary:KFT DIP-7X7")
+    )
+  )
